Commit message: tmp

File: urdf/balance_robot.xacro (robot description, xacro)
@@ -8,4 +8,5 @@
   <inertial>
     <origin rpy="0 0 0" xyz="4.1684108266638076e-05 0.000497123586462592 0.1077879171161801"/>
+    <!-- initial mass -> mass value="3.047016939610255"/-->
     <mass value="3.047016939610255"/>
     <inertia ixx="0.013885" ixy="0.0" ixz="-5e-06" iyy="0.0102" iyz="1.2e-05" izz="0.00539"/>
@@ -25,5 +26,5 @@
   </collision>
 </link>
-<link name="left_wheel_2">
+<link name="left_wheel">
   <inertial>
     <origin rpy="0 0 0" xyz="5.232905343968532e-16 0.013499725279272082 -6.175615574477433e-16"/>
@@ -45,5 +46,5 @@
   </collision>
 </link>
-<link name="right_wheel_1">
+<link name="right_wheel">
   <inertial>
     <origin rpy="0 0 0" xyz="2.0930055342611735e-15 -0.013500274720727637 6.661338147750939e-16"/>
@@ -73,7 +74,7 @@
   <origin rpy="0 0 0" xyz="0.0 0.077266 0.03301"/>
   <parent link="base_link"/>
-  <child link="left_wheel_2"/>
-  <axis xyz="-0.0 1.0 -0.0"/>
-  <limit velocity="12.0" effort="0.4"/>
+  <child link="left_wheel"/>
+  <axis xyz="0.0 1.0 0.0"/>
+  <limit velocity="10.47" effort="1.5"/> <!-- vel->rad/s effort->N*m -->
   <dynamics damping="0.1"/>
 </joint>
@@ -81,7 +82,7 @@
   <origin rpy="0 0 0" xyz="0.0 -0.078734 0.03301"/>
   <parent link="base_link"/>
-  <child link="right_wheel_1"/>
+  <child link="right_wheel"/>
   <axis xyz="0.0 1.0 0.0"/>
-  <limit velocity="12.0" effort="0.4"/>
+  <limit velocity="10.47" effort="1.5"/> <!-- vel->rad/s effort->N*m -->
   <dynamics damping="0.1"/>
 </joint>

Commit message: Add imu_sensor

File: urdf/balance_robot.xacro (robot description, xacro)
@@ -26,4 +26,5 @@
   </collision>
 </link>
+<link name="imu_link"/>
 <link name="left_wheel">
   <inertial>
@@ -71,4 +72,9 @@
   <origin rpy="0 0 0" xyz="0 0 0"/>
 </joint>
+<joint name="imu_joint" type="fixed">
+  <parent link = "base_link"/>
+  <child link = "imu_link"/>
+  <origin rpy="0 0 0" xyz="0 0 0.150"/>
+</joint>
 <joint name="left_wheel_joint" type="continuous">
   <origin rpy="0 0 0" xyz="0.0 0.077266 0.03301"/>

Commit message: Add calc param script

File: urdf/balance_robot.xacro (robot description, xacro)
@@ -7,8 +7,8 @@
 <link name="body_link">
   <inertial>
-    <origin rpy="0 0 0" xyz="4.1684108266638076e-05 0.000497123586462592 0.1077879171161801"/>
+    <origin rpy="0 0 0" xyz="0 0 0.10"/>
     <!-- initial mass -> mass value="3.047016939610255"/-->
-    <mass value="3.047016939610255"/>
-    <inertia ixx="0.013885" ixy="0.0" ixz="-5e-06" iyy="0.0102" iyz="1.2e-05" izz="0.00539"/>
+    <mass value="0.8"/>
+    <inertia ixx="0.003013" ixy="0.0" ixz="0.0" iyy="0.00194667" iyz="0.0" izz="0.00154667"/>
   </inertial>
   <visual>
@@ -30,6 +30,7 @@
   <inertial>
     <origin rpy="0 0 0" xyz="5.232905343968532e-16 0.013499725279272082 -6.175615574477433e-16"/>
-    <mass value="0.700600998578198"/>
-    <inertia ixx="0.000227" ixy="0.0" ixz="0.0" iyy="0.000369" iyz="-0.0" izz="0.000227"/>
+    <!-- initial mass -> mass value="0.700600998578198"/-->
+    <mass value="0.05"/>
+    <inertia ixx="0.0000541667" ixy="0.0" ixz="0.0" iyy="0.000105625" iyz="0.0" izz="0.0000541667"/>
   </inertial>
   <visual>
@@ -50,6 +51,7 @@
   <inertial>
     <origin rpy="0 0 0" xyz="2.0930055342611735e-15 -0.013500274720727637 6.661338147750939e-16"/>
-    <mass value="0.700600998578198"/>
-    <inertia ixx="0.000227" ixy="-0.0" ixz="-0.0" iyy="0.000369" iyz="-0.0" izz="0.000227"/>
+    <!-- initial mass -> mass value="0.700600998578198"/-->
+    <mass value="0.05"/>
+    <inertia ixx="0.0000541667" ixy="0.0" ixz="0.0" iyy="0.000105625" iyz="0.0" izz="0.0000541667"/>
   </inertial>
   <visual>
@@ -82,5 +84,5 @@
   <child link="left_wheel"/>
   <axis xyz="0.0 1.0 0.0"/>
-  <limit velocity="10.47" effort="1.5"/> <!-- vel->rad/s effort->N*m -->
+  <limit velocity="11.52" effort="1.47"/> <!-- vel -> rad/s, effort -> N*m -->
   <dynamics damping="0.1"/>
 </joint>
@@ -90,5 +92,5 @@
   <child link="right_wheel"/>
   <axis xyz="0.0 1.0 0.0"/>
-  <limit velocity="10.47" effort="1.5"/> <!-- vel->rad/s effort->N*m -->
+  <limit velocity="11.52" effort="1.47"/> <!-- vel -> rad/s, effort -> N*m -->
   <dynamics damping="0.1"/>
 </joint>
