Commit message: modified model bug

File: urdf/bug_balance_robot_simple.urdf.xacro (robot description, xacro)
@@ -3,25 +3,23 @@
 <xacro:include filename="$(find balance_robot_description)/urdf/materials.xacro" />
 <xacro:include filename="$(find balance_robot_description)/urdf/balance_robot.trans" />
-<xacro:include filename="$(find balance_robot_description)/urdf/balance_robot_simple.gazebo" />
+<xacro:include filename="$(find balance_robot_description)/urdf/balance_robot.gazebo" />
 <xacro:property name="PI" value="3.14159"/>
-<xacro:property name="PI_2" value="1.57079"/>
-<link name="base_footprint"/>
+<link name="base_link"/>
 <joint name="base_joint" type="fixed">
-  <parent link = "base_footprint"/>
-  <child link = "base_link"/>>
-  <origin rpy="0 0 0" xyz="0 0 0"/>
+  <parent link = "base_link"/>
+  <child link = "body_link"/>
+  <!--<origin rpy="0 0 0" xyz="0 0 0"/>-->
+  <origin rpy="0 0 0" xyz="0 0 0.0325"/>
 </joint>
-<link name="base_link">
+<link name="body_link">
   <inertial>
     <origin rpy="0 0 0" xyz="0 0 0.0786"/>
     <mass value="0.926999"/>
-    <inertia ixx="5.762E-03" ixy="1.926125E-06" ixz="-4.80363E-06"
-             iyy="4.501E-03" iyz="4.347E-05"
-             izz="1.818E-03"/>
+    <inertia ixx="5.762E-03" ixy="1.926125E-06" ixz="-4.80363E-06" iyy="4.501E-03" iyz="4.347E-05" izz="1.818E-03"/>
   </inertial>
   <visual>
     <origin rpy="0 0 0" xyz="0 0 0"/>
     <geometry>
-      <mesh filename="package://balance_robot_description/meshes/base_link_simple_body.stl" scale="0.001 0.001 0.001"/>
+      <mesh filename="package://balance_robot_description/meshes/base_link_simple_body_origin.stl" scale="0.001 0.001 0.001"/>
     </geometry>
     <material name="silver"/>
@@ -30,10 +28,10 @@
     <origin rpy="0 0 0" xyz="0 0 0"/>
     <geometry>
-      <mesh filename="package://balance_robot_description/meshes/base_link_simple_body.stl" scale="0.001 0.001 0.001"/>
+      <mesh filename="package://balance_robot_description/meshes/base_link_simple_body_origin.stl" scale="0.001 0.001 0.001"/>
     </geometry>
   </collision>
 </link>
 <joint name="imu_joint" type="fixed">
-  <parent link = "base_link"/>
+  <parent link = "body_link"/>
   <child link = "imu_link"/>
   <origin rpy="0 0 0" xyz="0 0 0.145"/>
@@ -41,17 +39,44 @@
 <link name="imu_link"/>
 <joint name="left_wheel_joint" type="continuous">
-  <parent link="base_link"/>
+  <parent link="body_link"/>
   <child link="left_wheel"/>
-  <origin rpy="0 0 ${PI}" xyz="0.0 -0.081 0.0325"/>
+  <origin rpy="0 0 ${PI}" xyz="0.0 -0.081 0.0"/>
   <axis xyz="0.0 1.0 0.0"/>
   <limit velocity="10.47" effort="1.5"/> <!-- vel->rad/s effort->N*m -->
+  <dynamics damping="0.1"/>
 </joint>
 <link name="left_wheel">
   <inertial>
-    <origin rpy="0 0 0" xyz="0 -0.0114 0"/>
+    <origin rpy="0 0 0" xyz="0.0 -0.0114 0.0"/>
     <mass value="0.048361"/>
-    <inertia ixx="1.679E-05" ixy="0.0" ixz="0.0"
-             iyy="2.615E-05" iyz="-0.0"
-             izz="1.679E-05"/>
+    <inertia ixx="1.679E-05" ixy="0.0" ixz="0.0" iyy="2.615E-05" iyz="-0.0" izz="1.679E-05"/>
+  </inertial>
+  <visual>
+    <origin rpy="0 0 0" xyz="0 0 0.0"/>
+    <geometry>
+      <mesh filename="package://balance_robot_description/meshes/wheel_tire_simple_origin.stl" scale="0.001 0.001 0.001"/>
+    </geometry>
+    <material name="silver"/>
+  </visual>
+  <collision>
+    <origin rpy="0 0 0" xyz="0 0 0"/>
+    <geometry>
+      <mesh filename="package://balance_robot_description/meshes/wheel_tire_simple_origin.stl" scale="0.001 0.001 0.001"/>
+    </geometry>
+  </collision>
+</link>
+<joint name="right_wheel_joint" type="continuous">
+  <origin rpy="0 0 0" xyz="0.0 0.081 0.0"/>
+  <parent link="body_link"/>
+  <child link="right_wheel"/>
+  <axis xyz="0.0 1.0 0.0"/>
+  <limit velocity="10.47" effort="1.5"/>
+  <dynamics damping="0.1"/>
+</joint>
+<link name="right_wheel">
+  <inertial>
+    <origin rpy="0 0 0" xyz="0.0 0.0114 0.0"/>
+    <mass value="0.048361"/>
+    <inertia ixx="1.679E-05" ixy="0.0" ixz="0.0" iyy="2.615E-05" iyz="-0.0" izz="1.679E-05"/>
   </inertial>
   <visual>
@@ -69,32 +94,3 @@
   </collision>
 </link>
-<joint name="right_wheel_joint" type="continuous">
-  <parent link="base_link"/>
-  <child link="right_wheel"/>
-  <origin rpy="0 0 0" xyz="0.0 0.081 0.0325"/>
-  <axis xyz="0.0 1.0 0.0"/>
-  <limit velocity="10.47" effort="1.5"/>
-</joint>
-<link name="right_wheel">
-  <inertial>
-    <origin rpy="0 0 0" xyz="0 0.0114 0"/>
-    <mass value="0.048361"/>
-    <inertia ixx="1.679E-05" ixy="0.0" ixz="0.0"
-             iyy="2.615E-05" iyz="-0.0"
-             izz="1.679E-05"/>
-  </inertial>
-  <visual>
-    <origin rpy="0 0 0" xyz="0 0 0"/>
-    <geometry>
-      <mesh filename="package://balance_robot_description/meshes/wheel_tire_simple_origin.stl" scale="0.001 0.001 0.001"/>
-    </geometry>
-    <material name="silver"/>
-  </visual>
-  <collision>
-    <origin rpy="0 0 0" xyz="0 0 0"/>
-    <geometry>
-      <mesh filename="package://balance_robot_description/meshes/wheel_tire_simple_origin.stl" scale="0.001 0.001 0.001"/>"/>
-    </geometry>
-  </collision>
-</link>
 </robot>
