Commit message: update mass params

File: urdf/balance_robot_simple.urdf.xacro (robot description, xacro)
@@ -8,9 +8,7 @@
 <link name="body_link">
   <inertial>
-    <!-- temp -->
-    <origin rpy="0 0 0" xyz="4.1684108266638076e-05 0.000497123586462592 0.1077879171161801"/>
-    <!-- initial mass -> mass value="3.047016939610255"/-->
-    <mass value="3.047016939610255"/>
-    <inertia ixx="0.013885" ixy="0.0" ixz="-5e-06" iyy="0.0102" iyz="1.2e-05" izz="0.00539"/>
+    <origin rpy="0 0 0" xyz="0 0 0"/>
+    <mass value="0,926999"/>
+    <inertia ixx="1.149e-2" ixy="1.99915e-06" ixz="-1.001e-06" iyy="1.023e-02" iyz="-6.657e-05" izz="1.820e-03"/>
   </inertial>
   <visual>
@@ -32,7 +30,7 @@
   <inertial>
     <!-- temp -->
-    <origin rpy="0 0 0" xyz="5.232905343968532e-16 0.013499725279272082 -6.175615574477433e-16"/>
-    <mass value="0.700600998578198"/>
-    <inertia ixx="0.000227" ixy="0.0" ixz="0.0" iyy="0.000369" iyz="-0.0" izz="0.000227"/>
+    <origin origin rpy="0 0 ${PI}" xyz="0.0 -0.081 0.0"/>
+    <mass value="0.048361"/>
+    <inertia ixx="2.305e-05" ixy="0.0" ixz="0.0" iyy="2.615e-05" iyz="-0.0" izz="2.305e-05"/>
   </inertial>
   <visual>
@@ -52,8 +50,7 @@
 <link name="right_wheel">
   <inertial>
-    <!-- temp -->
-    <origin rpy="0 0 0" xyz="2.0930055342611735e-15 -0.013500274720727637 6.661338147750939e-16"/>
-    <mass value="0.700600998578198"/>
-    <inertia ixx="0.000227" ixy="-0.0" ixz="-0.0" iyy="0.000369" iyz="-0.0" izz="0.000227"/>
+    <origin rpy="0 0 ${PI}" xyz="0.0 0.081 0.0"/>
+    <mass value="0.048361"/>
+    <inertia ixx="2.305e-05" ixy="0.0" ixz="0.0" iyy="2.615e-05" iyz="-0.0" izz="2.305e-05"/>
   </inertial>
   <visual>

Commit message: シンプルモデルのgazebo出力化及びReadme変更

File: urdf/balance_robot_simple.urdf.xacro (robot description, xacro)
@@ -9,5 +9,5 @@
   <inertial>
     <origin rpy="0 0 0" xyz="0 0 0"/>
-    <mass value="0,926999"/>
+    <mass value="0.926999"/>
     <inertia ixx="1.149e-2" ixy="1.99915e-06" ixz="-1.001e-06" iyy="1.023e-02" iyz="-6.657e-05" izz="1.820e-03"/>
   </inertial>
@@ -29,6 +29,5 @@
 <link name="left_wheel">
   <inertial>
-    <!-- temp -->
-    <origin origin rpy="0 0 ${PI}" xyz="0.0 -0.081 0.0"/>
+    <origin rpy="0 0 ${PI}" xyz="0.0 -0.081 0.0"/>
     <mass value="0.048361"/>
     <inertia ixx="2.305e-05" ixy="0.0" ixz="0.0" iyy="2.615e-05" iyz="-0.0" izz="2.305e-05"/>

Commit message: temp commit

File: urdf/balance_robot_simple.urdf.xacro (robot description, xacro)
@@ -9,4 +9,5 @@
   <inertial>
     <origin rpy="0 0 0" xyz="0 0 0"/>
+    <!--<origin rpy="0 0 0" xyz="0 0 0.0325"/>-->
     <mass value="0.926999"/>
     <inertia ixx="1.149e-2" ixy="1.99915e-06" ixz="-1.001e-06" iyy="1.023e-02" iyz="-6.657e-05" izz="1.820e-03"/>
@@ -14,4 +15,5 @@
   <visual>
     <origin rpy="0 0 0" xyz="0 0 0"/>
+    <!--<origin rpy="0 0 0" xyz="0 0 0.0325"/>-->
     <geometry>
       <mesh filename="package://balance_robot_description/meshes/base_link_simple_body_origin.stl" scale="0.001 0.001 0.001"/>
@@ -21,4 +23,5 @@
   <collision>
     <origin rpy="0 0 0" xyz="0 0 0"/>
+    <!--<origin rpy="0 0 0" xyz="0 0 0.0325"/>-->
     <geometry>
       <mesh filename="package://balance_robot_description/meshes/base_link_simple_body_origin.stl" scale="0.001 0.001 0.001"/>
@@ -34,5 +37,6 @@
   </inertial>
   <visual>
-    <origin rpy="0 0 0" xyz="0 0 0"/>
+    <!--<origin rpy="0 0 ${PI}" xyz="0.0 -0.081 0.0325"/>-->
+    <origin rpy="0 0 0" xyz="0 0 0.0"/>
     <geometry>
       <mesh filename="package://balance_robot_description/meshes/wheel_tire_simple_origin.stl" scale="0.001 0.001 0.001"/>
@@ -41,4 +45,5 @@
   </visual>
   <collision>
+    <!--<origin rpy="0 0 ${PI}" xyz="0.0 -0.081 0.0"/>-->
     <origin rpy="0 0 0" xyz="0 0 0"/>
     <geometry>
@@ -47,4 +52,5 @@
   </collision>
 </link>
+<!--
 <link name="right_wheel">
   <inertial>
@@ -67,17 +73,20 @@
   </collision>
 </link>
+-->
 <joint name="base_joint" type="fixed">
   <parent link = "base_link"/>
   <child link = "body_link"/>
-  <origin rpy="0 0 0" xyz="0 0 0"/>
+  <!--<origin rpy="0 0 0" xyz="0 0 0"/>-->
+  <origin rpy="0 0 0" xyz="0 0 0.0325"/>
 </joint>
 <joint name="imu_joint" type="fixed">
-  <parent link = "base_link"/>
+  <parent link = "body_link"/>
   <child link = "imu_link"/>
   <origin rpy="0 0 0" xyz="0 0 0.145"/>
 </joint>
 <joint name="left_wheel_joint" type="continuous">
+  <!--<origin rpy="0 0 ${PI}" xyz="0.0 -0.081 0.0"/>-->
   <origin rpy="0 0 ${PI}" xyz="0.0 -0.081 0.0"/>
-  <parent link="base_link"/>
+  <parent link="body_link"/>
   <child link="left_wheel"/>
   <axis xyz="0.0 1.0 0.0"/>
@@ -85,11 +94,13 @@
   <dynamics damping="0.1"/>
 </joint>
+<!--
 <joint name="right_wheel_joint" type="continuous">
   <origin rpy="0 0 0" xyz="0.0 0.081 0.0"/>
-  <parent link="base_link"/>
+  <parent link="body_link"/>
   <child link="right_wheel"/>
   <axis xyz="0.0 1.0 0.0"/>
-  <limit velocity="10.47" effort="1.5"/> <!-- vel->rad/s effort->N*m -->
+  <limit velocity="10.47" effort="1.5"/>
   <dynamics damping="0.1"/>
 </joint>
+-->
 </robot>

Commit message: temp 2

File: urdf/balance_robot_simple.urdf.xacro (robot description, xacro)
@@ -30,4 +30,13 @@
 </link>
 <link name="imu_link"/>
+<joint name="left_wheel_joint" type="continuous">
+  <parent link="body_link"/>
+  <child link="left_wheel"/>
+  <!--<origin rpy="0 0 ${PI}" xyz="0.0 -0.081 0.0"/>-->
+  <origin rpy="0 0 ${PI}" xyz="0.0 -0.081 0.0"/>
+  <axis xyz="0.0 1.0 0.0"/>
+  <limit velocity="10.47" effort="1.5"/> <!-- vel->rad/s effort->N*m -->
+  <dynamics damping="0.1"/>
+</joint>
 <link name="left_wheel">
   <inertial>
@@ -52,5 +61,4 @@
   </collision>
 </link>
-<!--
 <link name="right_wheel">
   <inertial>
@@ -73,5 +81,4 @@
   </collision>
 </link>
--->
 <joint name="base_joint" type="fixed">
   <parent link = "base_link"/>
@@ -85,14 +92,4 @@
   <origin rpy="0 0 0" xyz="0 0 0.145"/>
 </joint>
-<joint name="left_wheel_joint" type="continuous">
-  <!--<origin rpy="0 0 ${PI}" xyz="0.0 -0.081 0.0"/>-->
-  <origin rpy="0 0 ${PI}" xyz="0.0 -0.081 0.0"/>
-  <parent link="body_link"/>
-  <child link="left_wheel"/>
-  <axis xyz="0.0 1.0 0.0"/>
-  <limit velocity="10.47" effort="1.5"/> <!-- vel->rad/s effort->N*m -->
-  <dynamics damping="0.1"/>
-</joint>
-<!--
 <joint name="right_wheel_joint" type="continuous">
   <origin rpy="0 0 0" xyz="0.0 0.081 0.0"/>
@@ -103,4 +100,3 @@
   <dynamics damping="0.1"/>
 </joint>
--->
 </robot>

Commit message: バグでない状態

File: urdf/balance_robot_simple.urdf.xacro (robot description, xacro)
@@ -6,14 +6,18 @@
 <xacro:property name="PI" value="3.14159"/>
 <link name="base_link"/>
+<joint name="base_joint" type="fixed">
+  <parent link = "base_link"/>
+  <child link = "body_link"/>
+  <!--<origin rpy="0 0 0" xyz="0 0 0"/>-->
+  <origin rpy="0 0 0" xyz="0 0 0.0325"/>
+</joint>
 <link name="body_link">
   <inertial>
-    <origin rpy="0 0 0" xyz="0 0 0"/>
-    <!--<origin rpy="0 0 0" xyz="0 0 0.0325"/>-->
+    <origin rpy="0 0 0" xyz="0 0 0.0786"/>
     <mass value="0.926999"/>
-    <inertia ixx="1.149e-2" ixy="1.99915e-06" ixz="-1.001e-06" iyy="1.023e-02" iyz="-6.657e-05" izz="1.820e-03"/>
+    <inertia ixx="5.762E-03" ixy="1.926125E-06" ixz="-4.80363E-06" iyy="4.501E-03" iyz="4.347E-05" izz="1.818E-03"/>
   </inertial>
   <visual>
     <origin rpy="0 0 0" xyz="0 0 0"/>
-    <!--<origin rpy="0 0 0" xyz="0 0 0.0325"/>-->
     <geometry>
       <mesh filename="package://balance_robot_description/meshes/base_link_simple_body_origin.stl" scale="0.001 0.001 0.001"/>
@@ -23,5 +27,4 @@
   <collision>
     <origin rpy="0 0 0" xyz="0 0 0"/>
-    <!--<origin rpy="0 0 0" xyz="0 0 0.0325"/>-->
     <geometry>
       <mesh filename="package://balance_robot_description/meshes/base_link_simple_body_origin.stl" scale="0.001 0.001 0.001"/>
@@ -29,9 +32,13 @@
   </collision>
 </link>
+<joint name="imu_joint" type="fixed">
+  <parent link = "body_link"/>
+  <child link = "imu_link"/>
+  <origin rpy="0 0 0" xyz="0 0 0.145"/>
+</joint>
 <link name="imu_link"/>
 <joint name="left_wheel_joint" type="continuous">
   <parent link="body_link"/>
   <child link="left_wheel"/>
-  <!--<origin rpy="0 0 ${PI}" xyz="0.0 -0.081 0.0"/>-->
   <origin rpy="0 0 ${PI}" xyz="0.0 -0.081 0.0"/>
   <axis xyz="0.0 1.0 0.0"/>
@@ -41,10 +48,9 @@
 <link name="left_wheel">
   <inertial>
-    <origin rpy="0 0 ${PI}" xyz="0.0 -0.081 0.0"/>
+    <origin rpy="0 0 0" xyz="0.0 -0.0114 0.0"/>
     <mass value="0.048361"/>
-    <inertia ixx="2.305e-05" ixy="0.0" ixz="0.0" iyy="2.615e-05" iyz="-0.0" izz="2.305e-05"/>
+    <inertia ixx="1.679E-05" ixy="0.0" ixz="0.0" iyy="2.615E-05" iyz="-0.0" izz="1.679E-05"/>
   </inertial>
   <visual>
-    <!--<origin rpy="0 0 ${PI}" xyz="0.0 -0.081 0.0325"/>-->
     <origin rpy="0 0 0" xyz="0 0 0.0"/>
     <geometry>
@@ -54,5 +60,4 @@
   </visual>
   <collision>
-    <!--<origin rpy="0 0 ${PI}" xyz="0.0 -0.081 0.0"/>-->
     <origin rpy="0 0 0" xyz="0 0 0"/>
     <geometry>
@@ -61,9 +66,17 @@
   </collision>
 </link>
+<joint name="right_wheel_joint" type="continuous">
+  <origin rpy="0 0 0" xyz="0.0 0.081 0.0"/>
+  <parent link="body_link"/>
+  <child link="right_wheel"/>
+  <axis xyz="0.0 1.0 0.0"/>
+  <limit velocity="10.47" effort="1.5"/>
+  <dynamics damping="0.1"/>
+</joint>
 <link name="right_wheel">
   <inertial>
-    <origin rpy="0 0 ${PI}" xyz="0.0 0.081 0.0"/>
+    <origin rpy="0 0 0" xyz="0.0 0.0114 0.0"/>
     <mass value="0.048361"/>
-    <inertia ixx="2.305e-05" ixy="0.0" ixz="0.0" iyy="2.615e-05" iyz="-0.0" izz="2.305e-05"/>
+    <inertia ixx="1.679E-05" ixy="0.0" ixz="0.0" iyy="2.615E-05" iyz="-0.0" izz="1.679E-05"/>
   </inertial>
   <visual>
@@ -81,22 +94,3 @@
   </collision>
 </link>
-<joint name="base_joint" type="fixed">
-  <parent link = "base_link"/>
-  <child link = "body_link"/>
-  <!--<origin rpy="0 0 0" xyz="0 0 0"/>-->
-  <origin rpy="0 0 0" xyz="0 0 0.0325"/>
-</joint>
-<joint name="imu_joint" type="fixed">
-  <parent link = "body_link"/>
-  <child link = "imu_link"/>
-  <origin rpy="0 0 0" xyz="0 0 0.145"/>
-</joint>
-<joint name="right_wheel_joint" type="continuous">
-  <origin rpy="0 0 0" xyz="0.0 0.081 0.0"/>
-  <parent link="body_link"/>
-  <child link="right_wheel"/>
-  <axis xyz="0.0 1.0 0.0"/>
-  <limit velocity="10.47" effort="1.5"/>
-  <dynamics damping="0.1"/>
-</joint>
 </robot>

Commit message: change param & README

File: urdf/balance_robot_simple.urdf.xacro (robot description, xacro)
@@ -45,5 +45,6 @@
   <origin rpy="0 0 ${PI}" xyz="0.0 -0.081 0.0325"/>
   <axis xyz="0.0 1.0 0.0"/>
-  <limit velocity="10.47" effort="1.5"/> <!-- vel->rad/s effort->N*m -->
+  <limit velocity="11.5" effort="1.5"/> <!-- vel->rad/s effort->N*m -->
+  <!--dynamics friction="0.1" />-->
 </joint>
 <link name="left_wheel">
@@ -74,5 +75,6 @@
   <origin rpy="0 0 0" xyz="0.0 0.081 0.0325"/>
   <axis xyz="0.0 1.0 0.0"/>
-  <limit velocity="10.47" effort="1.5"/>
+  <limit velocity="11.5" effort="1.5"/>
+  <!--<dynamics friction="0.1" />-->
 </joint>
 <link name="right_wheel">

Commit message: correct wheel direction

File: urdf/balance_robot_simple.urdf.xacro (robot description, xacro)
@@ -43,5 +43,6 @@
   <parent link="base_link"/>
   <child link="left_wheel"/>
-  <origin rpy="0 0 ${PI}" xyz="0.0 -0.081 0.0325"/>
+  <origin rpy="0 0 0" xyz="0.0 -0.108 0.0325"/>
+  <!--<origin rpy="0 0 ${PI}" xyz="0.0 -0.081 0.0325"/>-->
   <axis xyz="0.0 1.0 0.0"/>
   <limit velocity="11.5" effort="1.5"/> <!-- vel->rad/s effort->N*m -->

Commit message: Change link direction

File: urdf/balance_robot_simple.urdf.xacro (robot description, xacro)
@@ -44,5 +44,5 @@
   <child link="left_wheel"/>
   <origin rpy="0 0 0" xyz="0.0 -0.108 0.0325"/>
-  <!--<origin rpy="0 0 ${PI}" xyz="0.0 -0.081 0.0325"/>-->
+  <!-- <origin rpy="0 0 ${PI}" xyz="0.0 -0.081 0.0325"/> -->
   <axis xyz="0.0 1.0 0.0"/>
   <limit velocity="11.5" effort="1.5"/> <!-- vel->rad/s effort->N*m -->
@@ -75,4 +75,5 @@
   <child link="right_wheel"/>
   <origin rpy="0 0 0" xyz="0.0 0.081 0.0325"/>
+  <!-- <origin rpy="0 0 ${PI}" xyz="0.0 0.108 0.0325"/> -->
   <axis xyz="0.0 1.0 0.0"/>
   <limit velocity="11.5" effort="1.5"/>
